File: docs/block-diagram.kicad_sch (KiCad schematic)
At the start: 0 parts

Commit message: release: v1.0.0
Other:
- note added: "UARTE TX P0.06"
- note added: "USB VCOM Serial Output"
- note added: "microSD Card Module CS: SD_CS MISO: 2kΩ series resistor"
- note removed: "microSD Card CS: SD_CS MISO: 2kΩ series resistor"
Changed lines of the file:
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@@
 	(generator "eeschema")
 	(generator_version "10.0")
-	(paper "User" 177.8 127)
+	(paper "User" 215.9 127)
 	(rectangle
-		(start 97.79 83.82)
-		(end 149.86 102.87)
+		(start 86.36 86.36)
+		(end 138.43 105.41)
 		(stroke
 			(width 0)
@@
 	)
 	(rectangle
-		(start 53.34 19.05)
-		(end 120.65 39.37)
+		(start 41.91 21.59)
+		(end 109.22 41.91)
 		(stroke
 			(width 0)
@@
 	)
 	(rectangle
-		(start 30.48 83.82)
-		(end 76.2 102.87)
+		(start 19.05 86.36)
+		(end 64.77 105.41)
 		(stroke
 			(width 0)
@@
 		)
 	)
-	(text "W5500\nEthernet Controller\nCS: W5500_CS"
+	(rectangle
+		(start 146.05 21.59)
+		(end 198.12 40.64)
+		(stroke
+			(width 0)
+			(type default)
+		)
+		(fill
+			(type none)
+		)
+	)
+	(text "USB VCOM\nSerial Output"
 		(exclude_from_sim no)
-		(at 52.07 93.98 0)
+		(at 170.18 31.75 0)
 		(effects
 			(font
@@
 		)
 	)
-	(text "microSD\nCard\nCS: SD_CS\nMISO: 2kΩ series resistor"
+	(text "W5500\nEthernet Controller\nCS: W5500_CS"
 		(exclude_from_sim no)
-		(at 123.19 93.98 0)
+		(at 40.64 96.52 0)
+		(effects
+			(font
+				(size 2.54 2.54)
+			)
+		)
+	)
+	(text "UARTE TX\nP0.06"
+		(exclude_from_sim no)
+		(at 130.81 30.48 0)
+		(effects
+			(font
+				(size 2.54 2.54)
+			)
+		)
+	)
+	(text "microSD Card Module\nCS: SD_CS\nMISO: 2kΩ series resistor"
+		(exclude_from_sim no)
+		(at 111.76 96.52 0)
 		(effects
 			(font
@@
 	(text "nRF52840 DK"
 		(exclude_from_sim no)
-		(at 86.36 30.48 0)
+		(at 74.93 33.02 0)
 		(effects
 			(font
@@
 	(text "Shared SPI Bus\nSCK / MOSI / MISO"
 		(exclude_from_sim no)
-		(at 87.63 57.15 0)
+		(at 76.2 59.69 0)
 		(effects
 			(font
@@
 	)
 	(junction
-		(at 86.36 71.12)
+		(at 74.93 73.66)
 		(diameter 0)
 		(color 0 0 0 0)
@@
 	(wire
 		(pts
-			(xy 86.36 39.37) (xy 86.36 52.07)
+			(xy 74.93 41.91) (xy 74.93 54.61)
 		)
 		(stroke
@@
 	(wire
 		(pts
-			(xy 53.34 71.12) (xy 86.36 71.12)
+			(xy 41.91 73.66) (xy 74.93 73.66)
 		)
 		(stroke
@@
 	(wire
 		(pts
-			(xy 86.36 71.12) (xy 120.65 71.12)
+			(xy 74.93 73.66) (xy 109.22 73.66)
 		)
 		(stroke
@@
 	(wire
 		(pts
-			(xy 53.34 71.12) (xy 53.34 83.82)
+			(xy 41.91 73.66) (xy 41.91 86.36)
 		)
 		(stroke
@@
 	(wire
 		(pts
-			(xy 120.65 71.12) (xy 120.65 83.82)
+			(xy 109.22 73.66) (xy 109.22 86.36)
 		)
 		(stroke
@@
 	(wire
 		(pts
-			(xy 86.36 62.23) (xy 86.36 71.12)
+			(xy 109.22 30.48) (xy 123.19 30.48)
 		)
 		(stroke
+			(width 0)
+			(type default)
+		)
+	)
+	(wire
+		(pts
+			(xy 139.7 30.48) (xy 146.05 30.48)
+		)
+		(stroke
+			(width 0)
+			(type default)
+		)
+	)
+	(wire
+		(pts
+			(xy 74.93 64.77) (xy 74.93 73.66)
+		)
+		(stroke
