File: docs/wiring.kicad_sch (KiCad schematic)
At the start: 4 parts, among them J1 Micro_SD_Card, U1 nRF52840, U2 W5500

Commit message: release: v1.0.0
Connections:
- net UARTE_TX: now reaches U1.L1 (P0.06)
Other:
- note added: "Onboard Debugger USB VCOM"
Changed lines of the file:
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@@
 	(generator_version "10.0")
 	(paper "User" 254 228.6)
+	(rectangle
+		(start 124.46 97.79)
+		(end 146.05 104.14)
+		(stroke
+			(width 0)
+			(type default)
+		)
+		(fill
+			(type none)
+		)
+	)
+	(text "Onboard Debugger\nUSB VCOM"
+		(exclude_from_sim no)
+		(at 135.89 101.6 0)
+		(effects
+			(font
+				(size 1.27 1.27)
+			)
+		)
+	)
 	(junction
 		(at 96.52 113.03)
@@
 	(wire
 		(pts
-			(xy 201.93 99.06) (xy 201.93 200.66)
+			(xy 201.93 105.41) (xy 201.93 200.66)
 		)
 		(stroke
@@
 	(wire
 		(pts
+			(xy 157.48 109.22) (xy 157.48 95.25)
+		)
+		(stroke
+			(width 0)
+			(type default)
+		)
+	)
+	(wire
+		(pts
 			(xy 101.6 95.25) (xy 101.6 104.14)
 		)
@@
 	(wire
 		(pts
-			(xy 171.45 102.87) (xy 171.45 115.57)
+			(xy 171.45 109.22) (xy 171.45 115.57)
 		)
 		(stroke
@@
 	(wire
 		(pts
-			(xy 181.61 97.79) (xy 167.64 97.79)
+			(xy 181.61 100.33) (xy 167.64 100.33)
 		)
 		(stroke
@@
 	(wire
 		(pts
+			(xy 106.68 100.33) (xy 124.46 100.33)
+		)
+		(stroke
+			(width 0)
+			(type default)
+		)
+	)
+	(wire
+		(pts
 			(xy 101.6 135.89) (xy 101.6 127)
 		)
@@
 	(wire
 		(pts
-			(xy 181.61 196.85) (xy 181.61 97.79)
-		)
-		(stroke
-			(width 0)
-			(type default)
-		)
-	)
-	(wire
-		(pts
-			(xy 167.64 97.79) (xy 167.64 95.25)
-		)
-		(stroke
-			(width 0)
-			(type default)
-		)
-	)
-	(wire
-		(pts
-			(xy 165.1 99.06) (xy 201.93 99.06)
+			(xy 181.61 196.85) (xy 181.61 100.33)
+		)
+		(stroke
+			(width 0)
+			(type default)
+		)
+	)
+	(wire
+		(pts
+			(xy 167.64 100.33) (xy 167.64 95.25)
+		)
+		(stroke
+			(width 0)
+			(type default)
+		)
+	)
+	(wire
+		(pts
+			(xy 165.1 105.41) (xy 201.93 105.41)
 		)
 		(stroke
@@
 	(wire
 		(pts
-			(xy 157.48 95.25) (xy 157.48 102.87)
-		)
-		(stroke
-			(width 0)
-			(type default)
-		)
-	)
-	(wire
-		(pts
 			(xy 234.95 68.58) (xy 226.06 64.77)
 		)
@@
 	(wire
 		(pts
-			(xy 165.1 95.25) (xy 165.1 99.06)
+			(xy 165.1 95.25) (xy 165.1 105.41)
 		)
 		(stroke
@@
 	(wire
 		(pts
+			(xy 157.48 109.22) (xy 171.45 109.22)
+		)
+		(stroke
+			(width 0)
+			(type default)
+		)
+	)
+	(wire
+		(pts
 			(xy 69.85 193.04) (xy 171.45 193.04)
 		)
@@
 	(wire
 		(pts
+			(xy 106.68 95.25) (xy 106.68 100.33)
+		)
+		(stroke
+			(width 0)
+			(type default)
+		)
+	)
+	(wire
+		(pts
 			(xy 99.06 119.38) (xy 99.06 135.89)
 		)
@@
 	(wire
 		(pts
-			(xy 157.48 102.87) (xy 171.45 102.87)
-		)
-		(stroke
-			(width 0)
-			(type default)
-		)
-	)
-	(wire
-		(pts
 			(xy 154.94 95.25) (xy 154.94 118.11)
 		)
@@
 		)
 	)
-	(label "SD_CS"
-		(at 107.95 130.81 0)
+	(label "UARTE_TX"
+		(at 109.22 100.33 0)
 		(effects
 			(font
@@
 	)
 	(label "W5500_CS"
-		(at 68.58 110.49 0)
+		(at 166.37 105.41 0)
 		(effects
 			(font
@@
 		(effects
 			(font
+				(size 1.27 1.27)
+			)
+			(justify left bottom)
+		)
+	)
+	(label "SD_CS"
+		(at 101.6 104.14 0)
+		(effects
+			(font
